Commit message: moveit

File: src/my_robot_description/urdf/arm.xacro (robot description, xacro)
@@ -9,4 +9,10 @@
             <material name="grey"/>
         </visual>
+        <collision>
+            <geometry>
+                <box size="0.4 0.4 0.1"/>
+            </geometry>
+            <origin xyz="0 0 0.05" rpy="0 0 0"/>
+        </collision>
     </link>
     <link name="shoulder_link">
@@ -18,4 +24,10 @@
             <material name="blue"/>
         </visual>
+        <collision>
+            <geometry>
+                <box size="0.2 0.2 0.5"/>
+            </geometry>
+            <origin xyz="0 0 0.25" rpy="0 0 0"/>
+        </collision>
     </link>
     <link name="arm_link">
@@ -27,4 +39,10 @@
             <material name="grey"/>
         </visual>
+        <collision>
+            <geometry>
+                <box size="0.1 0.1 0.6"/>
+            </geometry>
+            <origin xyz="0 0 0.3" rpy="0 0 0"/>
+        </collision>
     </link>
     <link name="elbow_link">
@@ -36,4 +54,10 @@
             <material name="blue"/>
         </visual>
+        <collision>
+            <geometry>
+                <box size="0.1 0.1 0.1"/>
+            </geometry>
+            <origin xyz="0 0 0.05" rpy="0 0 0"/>
+        </collision>
     </link>
     <link name="forearm_link">
@@ -45,4 +69,10 @@
             <material name="grey"/>
         </visual>
+        <collision>
+            <geometry>
+                <box size="0.1 0.1 0.5"/>
+            </geometry>
+            <origin xyz="0 0 0.25" rpy="0 0 0"/>
+        </collision>
     </link>
     <link name="wrist_link">
@@ -54,4 +84,10 @@
             <material name="blue"/>
         </visual>
+        <collision>
+            <geometry>
+                <box size="0.1 0.1 0.05"/>
+            </geometry>
+            <origin xyz="0 0 0.025" rpy="0 0 0"/>
+        </collision>
     </link>
     <link name="hand_link">
@@ -63,4 +99,10 @@
             <material name="grey"/>
         </visual>
+        <collision>
+            <geometry>
+                <box size="0.1 0.1 0.02"/>
+            </geometry>
+            <origin xyz="0 0 0.01" rpy="0 0 0"/>
+        </collision>
     </link>
     <link name="tool_link"/>

File: src/my_robot_description/urdf/common_properties.xacro (robot description, xacro)
@@ -7,3 +7,18 @@
         <color rgba="0.0 0.0 1.0 1"/>
     </material>
+    <material name="red">
+        <color rgba="1.0 0.0 0.0 1"/>
+    </material>
+    <material name="green">
+        <color rgba="0.0 1.0 0.0 1"/>
+    </material>
+    <material name="yellow">
+        <color rgba="1.0 1.0 0.0 1"/>
+    </material>
+    <material name="purple">
+        <color rgba="0.5 0.0 0.5 1"/>
+    </material>
+    <material name="orange">
+        <color rgba="1.0 0.5 0.0 1"/>
+    </material>
 </robot>

File: src/my_robot_description/urdf/my_robot.urdf.xacro (robot description, xacro)
@@ -3,3 +3,10 @@
     <xacro:include filename="common_properties.xacro" />
     <xacro:include filename="arm.xacro" />
+    <xacro:include filename="gripper.xacro" />
+    <!-- 把夹爪固定到机械臂末端的 tool_link 上 -->
+    <joint name="tool_gripper_joint" type="fixed">
+        <parent link="tool_link"/>
+        <child link="gripper_base_link"/>
+        <origin xyz="0 0 0.01" rpy="0 0 0"/>
+    </joint>
 </robot>
